File: nRF52840_breakout.sch (KiCad schematic (older format))
At the start: 31 parts, among them J1 MM8130-2600, U1 nRF52840, Y1 32.768kHz, Y2 32MHz

Commit message: custom footprint for coax connector with switch
Parts:
- AE1: footprint (none) -> custom_footprints:nRF52840_dk_antenna
- J1: footprint (none) -> custom_footprints:COAX_MM8130-2600
Changed lines of the file:
@@
 F 0 "J1" H 10550 3150 50  0000 L CNN
 F 1 "MM8130-2600" H 10450 3250 50  0000 L CNN
-F 2 "" H 10350 3050 50  0001 C CNN
+F 2 "custom_footprints:COAX_MM8130-2600" H 10350 3050 50  0001 C CNN
 F 3 " ~" H 10350 3050 50  0001 C CNN
 	1    10350 3150
@@
 F 0 "AE1" H 10130 2041 50  0000 L CNN
 F 1 "Antenna" H 10130 1950 50  0000 L CNN
-F 2 "" H 10050 2050 50  0001 C CNN
+F 2 "custom_footprints:nRF52840_dk_antenna" H 10050 2050 50  0001 C CNN
 F 3 "~" H 10050 2050 50  0001 C CNN
 	1    10050 2050

Commit message: changed crystal load capacitance according to component / minor changes
Parts:
- C1, C2: value 12pF -> 12.5pF; footprint (none) -> Capacitor_SMD:C_0805_2012Metric_Pad1.15x1.40mm_HandSolder
- C10, C11, C12, C15, C16, C17, C18, C19, C20, C21, C22, C3, C4, C5, C6, C7, C8, C9: footprint (none) -> Capacitor_SMD:C_0805_2012Metric_Pad1.15x1.40mm_HandSolder
- C13, C14: value 12pF -> 8pF; footprint (none) -> Capacitor_SMD:C_0805_2012Metric_Pad1.15x1.40mm_HandSolder
- L1, L2, L3, L4: footprint (none) -> Inductor_SMD:L_0805_2012Metric_Pad1.15x1.40mm_HandSolder
- Y1, Y2: footprint (none) -> Crystal:Crystal_SMD_3215-2Pin_3.2x1.5mm
Changed lines of the file:
@@
 F 0 "L4" V 9185 3250 50  0000 C CNN
 F 1 "3.9nH" V 9094 3250 50  0000 C CNN
-F 2 "" H 9000 3250 50  0001 C CNN
+F 2 "Inductor_SMD:L_0805_2012Metric_Pad1.15x1.40mm_HandSolder" H 9000 3250 50  0001 C CNN
 F 3 "~" H 9000 3250 50  0001 C CNN
 	1    9000 3250
@@
 F 0 "C17" H 8508 3304 50  0000 R CNN
 F 1 "1pF" H 8508 3395 50  0000 R CNN
-F 2 "" H 8600 3350 50  0001 C CNN
+F 2 "Capacitor_SMD:C_0805_2012Metric_Pad1.15x1.40mm_HandSolder" H 8600 3350 50  0001 C CNN
 F 3 "~" H 8600 3350 50  0001 C CNN
 	1    8600 3350
@@
 F 0 "C20" H 9208 3304 50  0000 R CNN
 F 1 "1pF" H 9208 3395 50  0000 R CNN
-F 2 "" H 9300 3350 50  0001 C CNN
+F 2 "Capacitor_SMD:C_0805_2012Metric_Pad1.15x1.40mm_HandSolder" H 9300 3350 50  0001 C CNN
 F 3 "~" H 9300 3350 50  0001 C CNN
 	1    9300 3350
@@
 F 0 "C21" H 9758 3304 50  0000 R CNN
 F 1 "N.C." H 9758 3395 50  0000 R CNN
-F 2 "" H 9850 3350 50  0001 C CNN
+F 2 "Capacitor_SMD:C_0805_2012Metric_Pad1.15x1.40mm_HandSolder" H 9850 3350 50  0001 C CNN
 F 3 "~" H 9850 3350 50  0001 C CNN
 	1    9850 3350
@@
 F 0 "C22" V 9721 2650 50  0000 C CNN
 F 1 "1.2pF" V 9812 2650 50  0000 C CNN
-F 2 "" H 9950 2650 50  0001 C CNN
+F 2 "Capacitor_SMD:C_0805_2012Metric_Pad1.15x1.40mm_HandSolder" H 9950 2650 50  0001 C CNN
 F 3 "~" H 9950 2650 50  0001 C CNN
 	1    9950 2650
@@
 F 0 "Y2" V 7746 1719 50  0000 R CNN
 F 1 "32MHz" V 7655 1719 50  0000 R CNN
-F 2 "" H 7700 1850 50  0001 C CNN
-F 3 "~" H 7700 1850 50  0001 C CNN
+F 2 "Crystal:Crystal_SMD_3215-2Pin_3.2x1.5mm" H 7700 1850 50  0001 C CNN
+F 3 " NX5032GA-32.000000MHZ-LN-CD-1 " H 7700 1850 50  0001 C CNN
 	1    7700 1850
 	0    1    -1   0
@@
 P 7950 1650
 F 0 "C13" V 7721 1650 50  0000 C CNN
-F 1 "12pF" V 7812 1650 50  0000 C CNN
-F 2 "" H 7950 1650 50  0001 C CNN
+F 1 "8pF" V 7812 1650 50  0000 C CNN
+F 2 "Capacitor_SMD:C_0805_2012Metric_Pad1.15x1.40mm_HandSolder" H 7950 1650 50  0001 C CNN
 F 3 "~" H 7950 1650 50  0001 C CNN
 	1    7950 1650
@@
 P 7950 2050
 F 0 "C14" V 7721 2050 50  0000 C CNN
-F 1 "12pF" V 7812 2050 50  0000 C CNN
-F 2 "" H 7950 2050 50  0001 C CNN
+F 1 "8pF" V 7812 2050 50  0000 C CNN
+F 2 "Capacitor_SMD:C_0805_2012Metric_Pad1.15x1.40mm_HandSolder" H 7950 2050 50  0001 C CNN
 F 3 "~" H 7950 2050 50  0001 C CNN
 	1    7950 2050
@@
 F 0 "C4" H 3942 2196 50  0000 L CNN
 F 1 "100nF" H 3942 2105 50  0000 L CNN
-F 2 "" H 3850 2150 50  0001 C CNN
+F 2 "Capacitor_SMD:C_0805_2012Metric_Pad1.15x1.40mm_HandSolder" H 3850 2150 50  0001 C CNN
 F 3 "~" H 3850 2150 50  0001 C CNN
 	1    3850 2150
@@
 F 0 "C6" H 4492 2196 50  0000 L CNN
 F 1 "1µF" H 4492 2105 50  0000 L CNN
-F 2 "" H 4400 2150 50  0001 C CNN
+F 2 "Capacitor_SMD:C_0805_2012Metric_Pad1.15x1.40mm_HandSolder" H 4400 2150 50  0001 C CNN
 F 3 "~" H 4400 2150 50  0001 C CNN
 	1    4400 2150
@@
 P 2100 1950
 F 0 "C1" V 1871 1950 50  0000 C CNN
-F 1 "12pF" V 1962 1950 50  0000 C CNN
-F 2 "" H 2100 1950 50  0001 C CNN
+F 1 "12.5pF" V 1962 1950 50  0000 C CNN
+F 2 "Capacitor_SMD:C_0805_2012Metric_Pad1.15x1.40mm_HandSolder" H 2100 1950 50  0001 C CNN
 F 3 "~" H 2100 1950 50  0001 C CNN
 	1    2100 1950
@@
 P 2100 2350
 F 0 "C2" V 1871 2350 50  0000 C CNN
-F 1 "12pF" V 1962 2350 50  0000 C CNN
-F 2 "" H 2100 2350 50  0001 C CNN
+F 1 "12.5pF" V 1962 2350 50  0000 C CNN
+F 2 "Capacitor_SMD:C_0805_2012Metric_Pad1.15x1.40mm_HandSolder" H 2100 2350 50  0001 C CNN
 F 3 "~" H 2100 2350 50  0001 C CNN
 	1    2100 2350
@@
 F 0 "Y1" V 2396 2019 50  0000 R CNN
 F 1 "32.768kHz" V 2305 2019 50  0000 R CNN
-F 2 "" H 2350 2150 50  0001 C CNN
-F 3 "~" H 2350 2150 50  0001 C CNN
+F 2 "Crystal:Crystal_SMD_3215-2Pin_3.2x1.5mm" H 2350 2150 50  0001 C CNN
+F 3 "FC-135 32.7680KA-A5" H 2350 2150 50  0001 C CNN
 	1    2350 2150
 	0    -1   -1   0
@@
 F 0 "C3" H 2892 4446 50  0000 L CNN
 F 1 "4.7µF" H 2892 4355 50  0000 L CNN
-F 2 "" H 2800 4400 50  0001 C CNN
+F 2 "Capacitor_SMD:C_0805_2012Metric_Pad1.15x1.40mm_HandSolder" H 2800 4400 50  0001 C CNN
 F 3 "~" H 2800 4400 50  0001 C CNN
 	1    2800 4400
@@
 F 0 "C5" H 4292 4696 50  0000 L CNN
 F 1 "4.7µF" H 4292 4605 50  0000 L CNN
-F 2 "" H 4200 4650 50  0001 C CNN
+F 2 "Capacitor_SMD:C_0805_2012Metric_Pad1.15x1.40mm_HandSolder" H 4200 4650 50  0001 C CNN
 F 3 "~" H 4200 4650 50  0001 C CNN
 	1    4200 4650
@@
 F 0 "L1" V 3850 4450 50  0000 C CNN
 F 1 "10µH" V 3950 4450 50  0000 C CNN
-F 2 "" H 4000 4450 50  0001 C CNN
+F 2 "Inductor_SMD:L_0805_2012Metric_Pad1.15x1.40mm_HandSolder" H 4000 4450 50  0001 C CNN
 F 3 "~" H 4000 4450 50  0001 C CNN
 	1    4000 4450
@@
 F 0 "C7" H 4692 5696 50  0000 L CNN
 F 1 "4.7µF" H 4692 5605 50  0000 L CNN
-F 2 "" H 4600 5650 50  0001 C CNN
+F 2 "Capacitor_SMD:C_0805_2012Metric_Pad1.15x1.40mm_HandSolder" H 4600 5650 50  0001 C CNN
 F 3 "~" H 4600 5650 50  0001 C CNN
 	1    4600 5650
@@
 F 0 "C10" H 6142 6346 50  0000 L CNN
 F 1 "100nF" H 6142 6255 50  0000 L CNN
-F 2 "" H 6050 6300 50  0001 C CNN
+F 2 "Capacitor_SMD:C_0805_2012Metric_Pad1.15x1.40mm_HandSolder" H 6050 6300 50  0001 C CNN
 F 3 "~" H 6050 6300 50  0001 C CNN
 	1    6050 6300
@@
 F 0 "C16" H 8292 4746 50  0000 L CNN
 F 1 "100nF" H 8292 4655 50  0000 L CNN
-F 2 "" H 8200 4700 50  0001 C CNN
+F 2 "Capacitor_SMD:C_0805_2012Metric_Pad1.15x1.40mm_HandSolder" H 8200 4700 50  0001 C CNN
 F 3 "~" H 8200 4700 50  0001 C CNN
 	1    8200 4700
@@
 F 0 "C15" H 8292 4046 50  0000 L CNN
 F 1 "820pF" H 8292 3955 50  0000 L CNN
-F 2 "" H 8200 4000 50  0001 C CNN
+F 2 "Capacitor_SMD:C_0805_2012Metric_Pad1.15x1.40mm_HandSolder" H 8200 4000 50  0001 C CNN
 F 3 "~" H 8200 4000 50  0001 C CNN
 	1    8200 4000
@@
 F 0 "C18" V 8471 2350 50  0000 C CNN
 F 1 "100pF" V 8562 2350 50  0000 C CNN
-F 2 "" H 8700 2350 50  0001 C CNN
+F 2 "Capacitor_SMD:C_0805_2012Metric_Pad1.15x1.40mm_HandSolder" H 8700 2350 50  0001 C CNN
 F 3 "~" H 8700 2350 50  0001 C CNN
 	1    8700 2350
@@
 F 0 "C19" V 8900 2550 50  0000 C CNN
 F 1 "N.C." V 8800 2550 50  0000 C CNN
-F 2 "" H 8700 2550 50  0001 C CNN
+F 2 "Capacitor_SMD:C_0805_2012Metric_Pad1.15x1.40mm_HandSolder" H 8700 2550 50  0001 C CNN
 F 3 "~" H 8700 2550 50  0001 C CNN
 	1    8700 2550
@@
 F 0 "C12" H 6892 1996 50  0000 L CNN
 F 1 "100nF" H 6892 1905 50  0000 L CNN
-F 2 "" H 6800 1950 50  0001 C CNN
+F 2 "Capacitor_SMD:C_0805_2012Metric_Pad1.15x1.40mm_HandSolder" H 6800 1950 50  0001 C CNN
 F 3 "~" H 6800 1950 50  0001 C CNN
 	1    6800 1950
@@
 F 0 "C11" H 6892 1196 50  0000 L CNN
 F 1 "N.C." H 6892 1105 50  0000 L CNN
-F 2 "" H 6800 1150 50  0001 C CNN
+F 2 "Capacitor_SMD:C_0805_2012Metric_Pad1.15x1.40mm_HandSolder" H 6800 1150 50  0001 C CNN
 F 3 "~" H 6800 1150 50  0001 C CNN
 	1    6800 1150
@@
 F 0 "C9" H 5792 1146 50  0000 L CNN
 F 1 "47nF" H 5792 1055 50  0000 L CNN
-F 2 "" H 5700 1100 50  0001 C CNN
+F 2 "Capacitor_SMD:C_0805_2012Metric_Pad1.15x1.40mm_HandSolder" H 5700 1100 50  0001 C CNN
 F 3 "~" H 5700 1100 50  0001 C CNN
 	1    5700 1100
@@
 F 0 "C8" H 5442 1146 50  0000 L CNN
 F 1 "1µF" H 5442 1055 50  0000 L CNN
-F 2 "" H 5350 1100 50  0001 C CNN
+F 2 "Capacitor_SMD:C_0805_2012Metric_Pad1.15x1.40mm_HandSolder" H 5350 1100 50  0001 C CNN
 F 3 "~" H 5350 1100 50  0001 C CNN
 	1    5350 1100
@@
 F 0 "L3" H 4747 1296 50  0000 L CNN
 F 1 "10µH" H 4747 1205 50  0000 L CNN
-F 2 "" H 4700 1250 50  0001 C CNN
+F 2 "Inductor_SMD:L_0805_2012Metric_Pad1.15x1.40mm_HandSolder" H 4700 1250 50  0001 C CNN
 F 3 "~" H 4700 1250 50  0001 C CNN
 	1    4700 1250
@@
 F 0 "L2" H 4748 996 50  0000 L CNN
 F 1 "15nH" H 4748 905 50  0000 L CNN
-F 2 "" H 4700 950 50  0001 C CNN
+F 2 "Inductor_SMD:L_0805_2012Metric_Pad1.15x1.40mm_HandSolder" H 4700 950 50  0001 C CNN
 F 3 "~" H 4700 950 50  0001 C CNN
 	1    4700 950

Commit message: switched nfc antenna connector
Parts:
- Y2: footprint Crystal:Crystal_SMD_3215-2Pin_3.2x1.5mm -> Crystal:Crystal_SMD_5032-2Pin_5.0x3.2mm_HandSoldering
Changed lines of the file:
@@
 F 0 "Y2" V 7746 1719 50  0000 R CNN
 F 1 "32MHz" V 7655 1719 50  0000 R CNN
-F 2 "Crystal:Crystal_SMD_3215-2Pin_3.2x1.5mm" H 7700 1850 50  0001 C CNN
+F 2 "Crystal:Crystal_SMD_5032-2Pin_5.0x3.2mm_HandSoldering" H 7700 1850 50  0001 C CNN
 F 3 " NX5032GA-32.000000MHZ-LN-CD-1 " H 7700 1850 50  0001 C CNN
 	1    7700 1850

Commit message: minor changes to schematic and layout
Parts:
- AE1: footprint custom_footprints:nRF52840_dk_antenna -> RF_Antenna:Texas_SWRA117D_2.4GHz_Right
Other:
- moved on the sheet: C1, C2, Y1
Changed lines of the file:
@@
 $Descr A4 11693 8268
 encoding utf-8
-Sheet 1 3
+Sheet 1 4
 Title "nRF52840_breakout"
 Date "2019-03-22"
@@
 F 0 "AE1" H 10130 2041 50  0000 L CNN
 F 1 "Antenna" H 10130 1950 50  0000 L CNN
-F 2 "custom_footprints:nRF52840_dk_antenna" H 10050 2050 50  0001 C CNN
+F 2 "RF_Antenna:Texas_SWRA117D_2.4GHz_Right" H 10050 2050 50  0001 C CNN
 F 3 "~" H 10050 2050 50  0001 C CNN
 	1    10050 2050
@@
 L Device:C_Small C1
 U 1 1 5C95647E
-P 2100 1950
-F 0 "C1" V 1871 1950 50  0000 C CNN
-F 1 "12.5pF" V 1962 1950 50  0000 C CNN
-F 2 "Capacitor_SMD:C_0805_2012Metric_Pad1.15x1.40mm_HandSolder" H 2100 1950 50  0001 C CNN
-F 3 "~" H 2100 1950 50  0001 C CNN
-	1    2100 1950
+P 2700 1950
+F 0 "C1" V 2471 1950 50  0000 C CNN
+F 1 "12.5pF" V 2562 1950 50  0000 C CNN
+F 2 "Capacitor_SMD:C_0805_2012Metric_Pad1.15x1.40mm_HandSolder" H 2700 1950 50  0001 C CNN
+F 3 "~" H 2700 1950 50  0001 C CNN
+	1    2700 1950
 	0    -1   1    0
 $EndComp
@@
 L Device:C_Small C2
 U 1 1 5C956485
-P 2100 2350
-F 0 "C2" V 1871 2350 50  0000 C CNN
-F 1 "12.5pF" V 1962 2350 50  0000 C CNN
-F 2 "Capacitor_SMD:C_0805_2012Metric_Pad1.15x1.40mm_HandSolder" H 2100 2350 50  0001 C CNN
-F 3 "~" H 2100 2350 50  0001 C CNN
-	1    2100 2350
+P 2700 2350
+F 0 "C2" V 2471 2350 50  0000 C CNN
+F 1 "12.5pF" V 2562 2350 50  0000 C CNN
+F 2 "Capacitor_SMD:C_0805_2012Metric_Pad1.15x1.40mm_HandSolder" H 2700 2350 50  0001 C CNN
+F 3 "~" H 2700 2350 50  0001 C CNN
+	1    2700 2350
 	0    -1   1    0
 $EndComp
 Wire Wire Line
-	2350 2350 2350 2300
-Wire Wire Line
-	2350 2350 2200 2350
-Connection ~ 2350 2350
-Wire Wire Line
-	2000 1950 1950 1950
-Wire Wire Line
-	1950 1950 1950 2350
-Wire Wire Line
-	1950 2350 2000 2350
-Wire Wire Line
-	1950 2350 1950 2400
-Connection ~ 1950 2350
+	2950 2350 2950 2300
+Wire Wire Line
+	2950 2350 2800 2350
+Wire Wire Line
+	2600 1950 2550 1950
+Wire Wire Line
+	2550 1950 2550 2350
+Wire Wire Line
+	2550 2350 2600 2350
+Wire Wire Line
+	2550 2350 2550 2400
+Connection ~ 2550 2350
 $Comp
 L power:GND #PWR01
 U 1 1 5C956499
-P 1950 2400
-F 0 "#PWR01" H 1950 2150 50  0001 C CNN
-F 1 "GND" H 1955 2227 50  0000 C CNN
-F 2 "" H 1950 2400 50  0001 C CNN
-F 3 "" H 1950 2400 50  0001 C CNN
-	1    1950 2400
+P 2550 2400
+F 0 "#PWR01" H 2550 2150 50  0001 C CNN
+F 1 "GND" H 2555 2227 50  0000 C CNN
+F 2 "" H 2550 2400 50  0001 C CNN
+F 3 "" H 2550 2400 50  0001 C CNN
+	1    2550 2400
 	1    0    0    -1
 $EndComp
@@
 Wire Wire Line
 	3400 3050 3400 2350
-Wire Wire Line
-	2350 2350 3400 2350
 $Comp
 L Device:Crystal Y1
 U 1 1 5C95D561
-P 2350 2150
-F 0 "Y1" V 2396 2019 50  0000 R CNN
-F 1 "32.768kHz" V 2305 2019 50  0000 R CNN
-F 2 "Crystal:Crystal_SMD_3215-2Pin_3.2x1.5mm" H 2350 2150 50  0001 C CNN
-F 3 "FC-135 32.7680KA-A5" H 2350 2150 50  0001 C CNN
-	1    2350 2150
+P 2950 2150
+F 0 "Y1" V 2996 2019 50  0000 R CNN
+F 1 "32.768kHz" V 2905 2019 50  0000 R CNN
+F 2 "Crystal:Crystal_SMD_3215-2Pin_3.2x1.5mm" H 2950 2150 50  0001 C CNN
+F 3 "FC-135 32.7680KA-A5" H 2950 2150 50  0001 C CNN
+	1    2950 2150
 	0    -1   -1   0
 $EndComp
 Wire Wire Line
-	2200 1950 2350 1950
-Wire Wire Line
-	2350 2000 2350 1950
-Connection ~ 2350 1950
-Wire Wire Line
-	2350 1950 3550 1950
+	2800 1950 2950 1950
+Wire Wire Line
+	2950 2000 2950 1950
 Text GLabel 4300 4150 0    50   Input ~ 0
 P0.12
@@
 	1    0    0    -1
 $EndComp
+Wire Wire Line
+	2950 1950 3550 1950
+Connection ~ 2950 1950
+Wire Wire Line
+	2950 2350 3400 2350
+Connection ~ 2950 2350
+$Sheet
+S 950  1650 750  200
+U 5C9D648D
+F0 "Todo" 50
+F1 "nRF52840_breakout_todo.sch" 50
+$EndSheet
 $EndSCHEMATC

Commit message: added som like version of the breakout
Parts:
- removed C1, C2: 12.5pF, Capacitor_SMD:C_0805_2012Metric_Pad1.15x1.40mm_HandSolder, symbol Device:C_Small
- removed J1: MM8130-2600, custom_footprints:COAX_MM8130-2600, symbol Connector:Conn_Coaxial_x2
- removed Y2: 32MHz, Crystal:Crystal_SMD_5032-2Pin_5.0x3.2mm_HandSoldering, symbol Device:Crystal
- added C25: NC, Capacitor_SMD:C_0402_1005Metric, symbol Device:C_Small
- added J1: MM8930_2620, custom_footprints:MM8930_2620, symbol Connector:Conn_Coaxial
- added R4: NC, Resistor_SMD:R_0402_1005Metric, symbol Device:R_Small
- added R5: 0R, Resistor_SMD:R_0402_1005Metric, symbol Device:R_Small
- added Y2: 32MHz-XRCGB32M000F1H00R0, Crystal:Crystal_SMD_2016-4Pin_2.0x1.6mm, symbol Device:Crystal_GND24_Small
- C10, C11, C12, C15, C16, C17, C18, C19, C20, C21, C22, C3, C4, C5, C6, C7, C8, C9: footprint Capacitor_SMD:C_0805_2012Metric_Pad1.15x1.40mm_HandSolder -> Capacitor_SMD:C_0402_1005Metric
- C13, C14: value 8pF -> 6pF; footprint Capacitor_SMD:C_0805_2012Metric_Pad1.15x1.40mm_HandSolder -> Capacitor_SMD:C_0402_1005Metric
- L1: value 10µH -> NC; footprint Inductor_SMD:L_0805_2012Metric_Pad1.15x1.40mm_HandSolder -> Inductor_SMD:L_0402_1005Metric
- L2, L3, L4: footprint Inductor_SMD:L_0805_2012Metric_Pad1.15x1.40mm_HandSolder -> Inductor_SMD:L_0402_1005Metric
- Y1: value 32.768kHz -> 32.768kHz-SIT1533AI-H4-DCC-32.768E; footprint Crystal:Crystal_SMD_3215-2Pin_3.2x1.5mm -> Crystal:Crystal_SMD_2012-2Pin_2.0x1.2mm
Connections:
- net labels added: VDDH
- wire segments 179 -> 177
Other:
- moved on the sheet: AE1, C22

Commit message: path selection/charging/bme680 sensor integration
Parts:
- added J7: Conn_Coaxial, custom_footprints:MM8930_2620, symbol Connector:Conn_Coaxial
- added R11, R12: 0R, Resistor_SMD:R_0402_1005Metric, symbol Device:R_Small
Connections:
- net GND: now also J7.2 (Ext)
- net at C20.2, C21.2, L4.1: now also C22.1, R11.2, R12.2; no longer J1.1 (In)
- net at C17.2, L4.2: now also J1.2 (Ext); no longer U1.H23 (ANT)
- new net: AE1.1 (A), R11.1
- new net: J1.1 (In), U1.H23 (ANT)
- new net: J7.1 (In), R12.1
Other:
- moved on the sheet: AE1, C17, C20, C21, J1, L4
Changed lines of the file:
@@
 L Device:L_Small L4
 U 1 1 5C923E84
-P 9000 3250
-F 0 "L4" V 9185 3250 50  0000 C CNN
-F 1 "3.9nH" V 9094 3250 50  0000 C CNN
-F 2 "Inductor_SMD:L_0402_1005Metric" H 9000 3250 50  0001 C CNN
-F 3 "~" H 9000 3250 50  0001 C CNN
-	1    9000 3250
+P 9350 3250
+F 0 "L4" V 9535 3250 50  0000 C CNN
+F 1 "3.9nH" V 9444 3250 50  0000 C CNN
+F 2 "Inductor_SMD:L_0402_1005Metric" H 9350 3250 50  0001 C CNN
+F 3 "~" H 9350 3250 50  0001 C CNN
+	1    9350 3250
 	0    1    -1   0
 $EndComp
@@
 L Device:C_Small C17
 U 1 1 5C923F77
-P 8600 3350
-F 0 "C17" H 8508 3304 50  0000 R CNN
-F 1 "1pF" H 8508 3395 50  0000 R CNN
-F 2 "Capacitor_SMD:C_0402_1005Metric" H 8600 3350 50  0001 C CNN
-F 3 "~" H 8600 3350 50  0001 C CNN
-	1    8600 3350
+P 8950 3350
+F 0 "C17" H 8858 3304 50  0000 R CNN
+F 1 "1pF" H 8858 3395 50  0000 R CNN
+F 2 "Capacitor_SMD:C_0402_1005Metric" H 8950 3350 50  0001 C CNN
+F 3 "~" H 8950 3350 50  0001 C CNN
+	1    8950 3350
 	-1   0    0    1
 $EndComp
@@
 L power:GND #PWR014
 U 1 1 5C924A30
-P 8600 3650
-F 0 "#PWR014" H 8600 3400 50  0001 C CNN
-F 1 "GND" H 8605 3477 50  0000 C CNN
-F 2 "" H 8600 3650 50  0001 C CNN
-F 3 "" H 8600 3650 50  0001 C CNN
-	1    8600 3650
+P 8950 3650
+F 0 "#PWR014" H 8950 3400 50  0001 C CNN
+F 1 "GND" H 8955 3477 50  0000 C CNN
+F 2 "" H 8950 3650 50  0001 C CNN
+F 3 "" H 8950 3650 50  0001 C CNN
+	1    8950 3650
 	-1   0    0    -1
 $EndComp
@@
 L Device:C_Small C20
 U 1 1 5C927D1D
-P 9300 3350
-F 0 "C20" H 9208 3304 50  0000 R CNN
-F 1 "1pF" H 9208 3395 50  0000 R CNN
-F 2 "Capacitor_SMD:C_0402_1005Metric" H 9300 3350 50  0001 C CNN
-F 3 "~" H 9300 3350 50  0001 C CNN
-	1    9300 3350
+P 9650 3350
+F 0 "C20" H 9558 3304 50  0000 R CNN
+F 1 "1pF" H 9558 3395 50  0000 R CNN
+F 2 "Capacitor_SMD:C_0402_1005Metric" H 9650 3350 50  0001 C CNN
+F 3 "~" H 9650 3350 50  0001 C CNN
+	1    9650 3350
 	-1   0    0    1
 $EndComp
 Wire Wire Line
-	9300 3450 9300 3650
-Connection ~ 9300 3250
-Text Notes 9950 3200 2    50   ~ 0
+	9650 3450 9650 3650
+Connection ~ 9650 3250
+Text Notes 10300 3200 2    50   ~ 0
 RF
 $Comp
 L Device:C_Small C21
 U 1 1 5C92A711
-P 9850 3350
-F 0 "C21" H 9758 3304 50  0000 R CNN
-F 1 "N.C." H 9758 3395 50  0000 R CNN
-F 2 "Capacitor_SMD:C_0402_1005Metric" H 9850 3350 50  0001 C CNN
-F 3 "~" H 9850 3350 50  0001 C CNN
-	1    9850 3350
+P 10200 3350
+F 0 "C21" H 10108 3304 50  0000 R CNN
+F 1 "N.C." H 10108 3395 50  0000 R CNN
+F 2 "Capacitor_SMD:C_0402_1005Metric" H 10200 3350 50  0001 C CNN
+F 3 "~" H 10200 3350 50  0001 C CNN
+	1    10200 3350
 	-1   0    0    1
 $EndComp
 Wire Wire Line
-	9850 3250 10150 3250
-Wire Wire Line
-	9850 3450 9850 3650
+	10200 3250 10500 3250
+Wire Wire Line
+	10200 3450 10200 3650
 $Comp
 L Device:C_Small C22
@@
 L Device:Antenna AE1
 U 1 1 5C93430F
-P 10350 2050
-F 0 "AE1" H 10430 2041 50  0000 L CNN
-F 1 "Antenna" H 10430 1950 50  0000 L CNN
-F 2 "RF_Antenna:Texas_SWRA117D_2.4GHz_Right" H 10350 2050 50  0001 C CNN
-F 3 "~" H 10350 2050 50  0001 C CNN
-	1    10350 2050
+P 10350 1800
+F 0 "AE1" H 10430 1791 50  0000 L CNN
+F 1 "Antenna" H 10430 1700 50  0000 L CNN
+F 2 "RF_Antenna:Texas_SWRA117D_2.4GHz_Right" H 10350 1800 50  0001 C CNN
+F 3 "~" H 10350 1800 50  0001 C CNN
+	1    10350 1800
 	-1   0    0    -1
 $EndComp
@@
 L power:GND #PWR016
 U 1 1 5C936B52
-P 9300 3650
-F 0 "#PWR016" H 9300 3400 50  0001 C CNN
-F 1 "GND" H 9305 3477 50  0000 C CNN
-F 2 "" H 9300 3650 50  0001 C CNN
-F 3 "" H 9300 3650 50  0001 C CNN
-	1    9300 3650
+P 9650 3650
+F 0 "#PWR016" H 9650 3400 50  0001 C CNN
+F 1 "GND" H 9655 3477 50  0000 C CNN
+F 2 "" H 9650 3650 50  0001 C CNN
+F 3 "" H 9650 3650 50  0001 C CNN
+	1    9650 3650
 	-1   0    0    -1
 $EndComp
@@
 L power:GND #PWR018
 U 1 1 5C936B97
-P 9850 3650
-F 0 "#PWR018" H 9850 3400 50  0001 C CNN
-F 1 "GND" H 9855 3477 50  0000 C CNN
-F 2 "" H 9850 3650 50  0001 C CNN
-F 3 "" H 9850 3650 50  0001 C CNN
-	1    9850 3650
+P 10200 3650
+F 0 "#PWR018" H 10200 3400 50  0001 C CNN
+F 1 "GND" H 10205 3477 50  0000 C CNN
+F 2 "" H 10200 3650 50  0001 C CNN
+F 3 "" H 10200 3650 50  0001 C CNN
+	1    10200 3650
 	-1   0    0    -1
 $EndComp
@@
 	7300 3450 7250 3450
 Wire Wire Line
-	8600 3450 8600 3550
-Wire Wire Line
-	7250 3250 8600 3250
-Wire Wire Line
-	8600 3250 8900 3250
-Connection ~ 8600 3250
-Wire Wire Line
-	9100 3250 9300 3250
-Wire Wire Line
-	9300 3250 9850 3250
-Connection ~ 9850 3250
+	8950 3450 8950 3550
+Wire Wire Line
+	8950 3250 9250 3250
+Wire Wire Line
+	9450 3250 9650 3250
+Wire Wire Line
+	9650 3250 10200 3250
+Connection ~ 10200 3250
 Wire Wire Line
 	10350 2650 10350 3050
@@
 	10350 2250 10350 2650
 Wire Wire Line
-	8600 3550 8200 3550
-Wire Wire Line
 	8200 3550 8200 3150
 Wire Wire Line
 	8200 3150 7250 3150
-Connection ~ 8600 3550
-Wire Wire Line
-	8600 3550 8600 3650
+Connection ~ 8950 3550
+Wire Wire Line
+	8950 3550 8950 3650
 Wire Wire Line
 	7250 2850 7400 2850
@@
 L Connector:Conn_Coaxial J1
 U 1 1 5CD5A531
-P 10350 3250
-F 0 "J1" H 10450 3134 50  0000 L CNN
-F 1 "MM8930_2620" H 10450 3225 50  0000 L CNN
-F 2 "custom_footprints:MM8930_2620" H 10350 3250 50  0001 C CNN
-F 3 " ~" H 10350 3250 50  0001 C CNN
-	1    10350 3250
+P 8650 3450
+F 0 "J1" H 8750 3334 50  0000 L CNN
+F 1 "MM8930_2620" H 8450 3150 50  0000 L CNN
+F 2 "custom_footprints:MM8930_2620" H 8650 3450 50  0001 C CNN
+F 3 " ~" H 8650 3450 50  0001 C CNN
+	1    8650 3450
 	1    0    0    1
 $EndComp
+$Comp
+L Device:R_Small R11
+U 1 1 5CC69485
+P 10350 2150
+F 0 "R11" H 10409 2196 50  0000 L CNN
+F 1 "0R" H 10409 2105 50  0000 L CNN
+F 2 "Resistor_SMD:R_0402_1005Metric" H 10350 2150 50  0001 C CNN
+F 3 "~" H 10350 2150 50  0001 C CNN
+	1    10350 2150
+	1    0    0    -1
+$EndComp
+Wire Wire Line
+	10350 2000 10350 2050
+$Comp
+L Device:R_Small R12
+U 1 1 5CC72038
+P 10500 2650
+F 0 "R12" V 10304 2650 50  0000 C CNN
+F 1 "0R" V 10395 2650 50  0000 C CNN
+F 2 "Resistor_SMD:R_0402_1005Metric" H 10500 2650 50  0001 C CNN
+F 3 "~" H 10500 2650 50  0001 C CNN
+	1    10500 2650
+	0    1    1    0
+$EndComp
+Wire Wire Line
+	10350 2650 10400 2650
+Wire Wire Line
+	10600 2650 10650 2650
+$Comp
+L Connector:Conn_Coaxial J7
+U 1 1 5CC8403F
+P 10850 2650
+F 0 "J7" H 10949 2626 50  0000 L CNN
+F 1 "Conn_Coaxial" H 10949 2535 50  0000 L CNN
+F 2 "custom_footprints:MM8930_2620" H 10850 2650 50  0001 C CNN
+F 3 " ~" H 10850 2650 50  0001 C CNN
+	1    10850 2650
+	1    0    0    -1
+$EndComp
+$Comp
+L power:GND #PWR023
+U 1 1 5CC84745
+P 10850 2900
+F 0 "#PWR023" H 10850 2650 50  0001 C CNN
+F 1 "GND" H 10855 2727 50  0000 C CNN
+F 2 "" H 10850 2900 50  0001 C CNN
+F 3 "" H 10850 2900 50  0001 C CNN
+	1    10850 2900
+	1    0    0    -1
+$EndComp
+Wire Wire Line
+	10850 2850 10850 2900
+Wire Wire Line
+	7250 3250 8000 3250
+Wire Wire Line
+	8000 3250 8000 3450
+Wire Wire Line
+	8000 3450 8450 3450
+Wire Wire Line
+	8200 3550 8950 3550
+Wire Wire Line
+	8650 3250 8950 3250
+Connection ~ 8950 3250
+Wire Wire Line
+	10500 3250 10500 3050
+Wire Wire Line
+	10500 3050 10350 3050
 $EndSCHEMATC
