File: nRF52840_breakout_connector.sch (KiCad schematic (older format))
At the start: 28 parts, among them J2 Conn_01x12, J3 Conn_01x12, J4 Conn_01x17, J5 FPC 0.5mm RA SMD, J6 Pin Header 2x5, 1.27, U2 USB_TYPE_C

Commit message: changed crystal load capacitance according to component / minor changes
Parts:
- C23, C24, C25, C26, C27, C28: footprint (none) -> Capacitor_SMD:C_0805_2012Metric_Pad1.15x1.40mm_HandSolder
- FB1, FB2, FB3: footprint (none) -> Inductor_SMD:L_0805_2012Metric_Pad1.15x1.40mm_HandSolder
- H1, H2, H3, H4: footprint (none) -> MountingHole:MountingHole_2.2mm_M2_Pad_Via
- J2, J3: footprint (none) -> Connector_PinHeader_2.54mm:PinHeader_1x12_P2.54mm_Vertical
- J4: footprint (none) -> Connector_PinHeader_2.54mm:PinHeader_1x17_P2.54mm_Vertical
- J6: footprint (none) -> Connector_PinHeader_1.27mm:PinHeader_2x05_P1.27mm_Vertical_SMD
- R1, R2, R3, R4: footprint (none) -> Resistor_SMD:R_0805_2012Metric_Pad1.15x1.40mm_HandSolder
- TP1, TP2, TP3, TP4: footprint (none) -> TestPoint:TestPoint_Pad_1.0x1.0mm
- U2: footprint (none) -> custom_footprints:USB_C_Receptacle_Amphenol_12401610E4-2A
Changed lines of the file:
@@
 F 0 "R2" V 2550 3600 50  0000 C CNN
 F 1 "5.1k" V 2625 3600 50  0000 C CNN
-F 2 "" H 2700 3600 50  0001 C CNN
+F 2 "Resistor_SMD:R_0805_2012Metric_Pad1.15x1.40mm_HandSolder" H 2700 3600 50  0001 C CNN
 F 3 "~" H 2700 3600 50  0001 C CNN
 	1    2700 3600
@@
 F 0 "R1" V 2690 3700 50  0000 C CNN
 F 1 "5.1k" V 2625 3700 50  0000 C CNN
-F 2 "" H 2550 3700 50  0001 C CNN
+F 2 "Resistor_SMD:R_0805_2012Metric_Pad1.15x1.40mm_HandSolder" H 2550 3700 50  0001 C CNN
 F 3 "~" H 2550 3700 50  0001 C CNN
 	1    2550 3700
@@
 F 0 "C24" H 2642 1496 50  0000 L CNN
 F 1 "10µF" H 2642 1405 50  0000 L CNN
-F 2 "" H 2550 1450 50  0001 C CNN
+F 2 "Capacitor_SMD:C_0805_2012Metric_Pad1.15x1.40mm_HandSolder" H 2550 1450 50  0001 C CNN
 F 3 "~" H 2550 1450 50  0001 C CNN
 	1    2550 1450
@@
 F 0 "C25" H 3042 1496 50  0000 L CNN
 F 1 "100nF" H 3042 1405 50  0000 L CNN
-F 2 "" H 2950 1450 50  0001 C CNN
+F 2 "Capacitor_SMD:C_0805_2012Metric_Pad1.15x1.40mm_HandSolder" H 2950 1450 50  0001 C CNN
 F 3 "~" H 2950 1450 50  0001 C CNN
 	1    2950 1450
@@
 F 0 "C26" H 3192 996 50  0000 L CNN
 F 1 "10µF" H 3192 905 50  0000 L CNN
-F 2 "" H 3100 950 50  0001 C CNN
+F 2 "Capacitor_SMD:C_0805_2012Metric_Pad1.15x1.40mm_HandSolder" H 3100 950 50  0001 C CNN
 F 3 "~" H 3100 950 50  0001 C CNN
 	1    3100 950
@@
 F 0 "C23" H 2542 996 50  0000 L CNN
 F 1 "10µF" H 2542 905 50  0000 L CNN
-F 2 "" H 2450 950 50  0001 C CNN
+F 2 "Capacitor_SMD:C_0805_2012Metric_Pad1.15x1.40mm_HandSolder" H 2450 950 50  0001 C CNN
 F 3 "~" H 2450 950 50  0001 C CNN
 	1    2450 950
@@
 F 0 "FB3" V 2563 850 50  0000 C CNN
 F 1 "120R/0.55A" V 2654 850 50  0000 C CNN
-F 2 "" V 2730 850 50  0001 C CNN
+F 2 "Inductor_SMD:L_0805_2012Metric_Pad1.15x1.40mm_HandSolder" V 2730 850 50  0001 C CNN
 F 3 "~" H 2800 850 50  0001 C CNN
 	1    2800 850
@@
 F 0 "TP2" H 3300 1050 50  0000 L CNN
 F 1 "VBUS_nRF" H 3300 950 50  0000 L CNN
-F 2 "" H 3450 850 50  0001 C CNN
+F 2 "TestPoint:TestPoint_Pad_1.0x1.0mm" H 3450 850 50  0001 C CNN
 F 3 "~" H 3450 850 50  0001 C CNN
 	1    3250 850
@@
 F 0 "TP1" H 2350 1050 50  0000 L CNN
 F 1 "VBUS_Raw" H 2350 950 50  0000 L CNN
-F 2 "" H 2500 850 50  0001 C CNN
+F 2 "TestPoint:TestPoint_Pad_1.0x1.0mm" H 2500 850 50  0001 C CNN
 F 3 "~" H 2500 850 50  0001 C CNN
 	1    2300 850
@@
 F 0 "FB2" H 800 3804 50  0000 R CNN
 F 1 "120R/0.55A" H 800 3895 50  0000 R CNN
-F 2 "" V 830 3850 50  0001 C CNN
+F 2 "Inductor_SMD:L_0805_2012Metric_Pad1.15x1.40mm_HandSolder" V 830 3850 50  0001 C CNN
 F 3 "~" H 900 3850 50  0001 C CNN
 	1    900  3850
@@
 F 0 "FB1" V 1000 3550 50  0000 R CNN
 F 1 "120R/0.55A" V 900 3750 50  0000 R CNN
-F 2 "" V 730 3500 50  0001 C CNN
+F 2 "Inductor_SMD:L_0805_2012Metric_Pad1.15x1.40mm_HandSolder" V 730 3500 50  0001 C CNN
 F 3 "~" H 800 3500 50  0001 C CNN
 	1    800  3500
@@
 F 0 "R3" V 4254 2700 50  0000 C CNN
 F 1 "22" V 4345 2700 50  0000 C CNN
-F 2 "" H 4450 2700 50  0001 C CNN
+F 2 "Resistor_SMD:R_0805_2012Metric_Pad1.15x1.40mm_HandSolder" H 4450 2700 50  0001 C CNN
 F 3 "~" H 4450 2700 50  0001 C CNN
 	1    4450 2700
@@
 F 0 "R4" V 4250 2900 50  0000 C CNN
 F 1 "22" V 4350 2900 50  0000 C CNN
-F 2 "" H 4450 2900 50  0001 C CNN
+F 2 "Resistor_SMD:R_0805_2012Metric_Pad1.15x1.40mm_HandSolder" H 4450 2900 50  0001 C CNN
 F 3 "~" H 4450 2900 50  0001 C CNN
 	1    4450 2900
@@
 F 0 "J6" H 8100 2117 50  0000 C CNN
 F 1 "Pin Header 2x5, 1.27" H 8100 2026 50  0000 C CNN
-F 2 "" H 8050 1700 50  0001 C CNN
+F 2 "Connector_PinHeader_1.27mm:PinHeader_2x05_P1.27mm_Vertical_SMD" H 8050 1700 50  0001 C CNN
 F 3 "~" H 8050 1700 50  0001 C CNN
 	1    8050 1700
@@
 F 0 "TP4" H 6100 1800 50  0000 L CNN
 F 1 "NFC2" H 6100 1700 50  0000 L CNN
-F 2 "" H 6250 1600 50  0001 C CNN
+F 2 "TestPoint:TestPoint_Pad_1.0x1.0mm" H 6250 1600 50  0001 C CNN
 F 3 "~" H 6250 1600 50  0001 C CNN
 	1    6050 1600
@@
 F 0 "TP3" H 6100 1600 50  0000 L CNN
 F 1 "NFC1" H 6100 1500 50  0000 L CNN
-F 2 "" H 6250 1400 50  0001 C CNN
+F 2 "TestPoint:TestPoint_Pad_1.0x1.0mm" H 6250 1400 50  0001 C CNN
 F 3 "~" H 6250 1400 50  0001 C CNN
 	1    6050 1400
@@
 F 0 "C27" H 5508 1104 50  0000 R CNN
 F 1 "CTUNE1" H 5508 1195 50  0000 R CNN
-F 2 "" H 5600 1150 50  0001 C CNN
+F 2 "Capacitor_SMD:C_0805_2012Metric_Pad1.15x1.40mm_HandSolder" H 5600 1150 50  0001 C CNN
 F 3 "~" H 5600 1150 50  0001 C CNN
 	1    5600 1150
@@
 F 0 "C28" H 5508 1754 50  0000 R CNN
 F 1 "CTUNE2" H 5508 1845 50  0000 R CNN
-F 2 "" H 5600 1800 50  0001 C CNN
+F 2 "Capacitor_SMD:C_0805_2012Metric_Pad1.15x1.40mm_HandSolder" H 5600 1800 50  0001 C CNN
 F 3 "~" H 5600 1800 50  0001 C CNN
 	1    5600 1800
@@
 F 0 "J2" H 1530 5242 50  0000 L CNN
 F 1 "Conn_01x12" H 1530 5151 50  0000 L CNN
-F 2 "" H 1450 5250 50  0001 C CNN
+F 2 "Connector_PinHeader_2.54mm:PinHeader_1x12_P2.54mm_Vertical" H 1450 5250 50  0001 C CNN
 F 3 "~" H 1450 5250 50  0001 C CNN
 	1    1450 5250
@@
 F 0 "J3" H 2730 5242 50  0000 L CNN
 F 1 "Conn_01x12" H 2730 5151 50  0000 L CNN
-F 2 "" H 2650 5250 50  0001 C CNN
+F 2 "Connector_PinHeader_2.54mm:PinHeader_1x12_P2.54mm_Vertical" H 2650 5250 50  0001 C CNN
 F 3 "~" H 2650 5250 50  0001 C CNN
 	1    2650 5250
@@
 F 0 "H1" H 5150 2646 50  0000 L CNN
 F 1 "MountingHole" H 5150 2555 50  0000 L CNN
-F 2 "" H 5050 2600 50  0001 C CNN
+F 2 "MountingHole:MountingHole_2.2mm_M2_Pad_Via" H 5050 2600 50  0001 C CNN
 F 3 "~" H 5050 2600 50  0001 C CNN
 	1    5050 2600
@@
 F 0 "H3" H 6400 2646 50  0000 L CNN
 F 1 "MountingHole" H 6400 2555 50  0000 L CNN
-F 2 "" H 6300 2600 50  0001 C CNN
+F 2 "MountingHole:MountingHole_2.2mm_M2_Pad_Via" H 6300 2600 50  0001 C CNN
 F 3 "~" H 6300 2600 50  0001 C CNN
 	1    6300 2600
@@
 F 0 "H2" H 5150 2946 50  0000 L CNN
 F 1 "MountingHole" H 5150 2855 50  0000 L CNN
-F 2 "" H 5050 2900 50  0001 C CNN
+F 2 "MountingHole:MountingHole_2.2mm_M2_Pad_Via" H 5050 2900 50  0001 C CNN
 F 3 "~" H 5050 2900 50  0001 C CNN
 	1    5050 2900
@@
 F 0 "H4" H 6400 2946 50  0000 L CNN
 F 1 "MountingHole" H 6400 2855 50  0000 L CNN
-F 2 "" H 6300 2900 50  0001 C CNN
+F 2 "MountingHole:MountingHole_2.2mm_M2_Pad_Via" H 6300 2900 50  0001 C CNN
 F 3 "~" H 6300 2900 50  0001 C CNN
 	1    6300 2900
@@
 U 1 1 5C966DF9
 P 1650 3150
-F 0 "U2" H 1625 4637 60  0000 C CNN
-F 1 "USB_TYPE_C" H 1625 4531 60  0000 C CNN
-F 2 "" H 1650 3150 60  0000 C CNN
+F 0 "U2" H 1650 4350 60  0000 C CNN
+F 1 "USB_TYPE_C" H 1650 4200 60  0000 C CNN
+F 2 "custom_footprints:USB_C_Receptacle_Amphenol_12401610E4-2A" H 1650 3150 60  0001 C CNN
 F 3 "" H 1650 3150 60  0000 C CNN
 	1    1650 3150
@@
 F 0 "J4" H 4180 5592 50  0000 L CNN
 F 1 "Conn_01x17" H 4180 5501 50  0000 L CNN
-F 2 "" H 4100 5550 50  0001 C CNN
+F 2 "Connector_PinHeader_2.54mm:PinHeader_1x17_P2.54mm_Vertical" H 4100 5550 50  0001 C CNN
 F 3 "~" H 4100 5550 50  0001 C CNN
 	1    4100 5550

Commit message: switched nfc antenna connector
Parts:
- removed J5: FPC 0.5mm RA SMD, symbol Connector_Generic:Conn_01x05
- added J?: 1734592-5, custom_footprints:CONNECTOR_FFC_1734592-5, symbol CONNECTOR_FFC_1734592-5:1734592-5
Connections:
- wire segments 94 -> 96
Changed lines of the file:
@@
 Wire Notes Line
 	9000 500  9000 2250
-$Comp
-L Connector_Generic:Conn_01x05 J?
-U 1 1 5C9538C5
-P 6400 1500
-AR Path="/5C9538C5" Ref="J?"  Part="1"
-AR Path="/5C94F379/5C9538C5" Ref="J5"  Part="1"
-F 0 "J5" H 6480 1542 50  0000 L CNN
-F 1 "FPC 0.5mm RA SMD" H 6480 1451 50  0000 L CNN
-F 2 "" H 6400 1500 50  0001 C CNN
-F 3 "~" H 6400 1500 50  0001 C CNN
-	1    6400 1500
-	1    0    0    -1
-$EndComp
 Text Notes 4850 600  0    50   ~ 0
 NFC Antenna Connector
@@
 NoConn ~ 950  2400
 NoConn ~ 950  2300
+$Comp
+L CONNECTOR_FFC_1734592-5:1734592-5 J?
+U 1 1 5C986751
+P 6600 1600
+F 0 "J?" H 6372 1646 50  0000 R CNN
+F 1 "1734592-5" H 6400 1550 50  0000 R CNN
+F 2 "custom_footprints:CONNECTOR_FFC_1734592-5" H 6600 1600 50  0001 L BNN
+F 3 "None" H 6600 1600 50  0001 L BNN
+F 4 "TE Connectivity" H 6600 1600 50  0001 L BNN "Field4"
+F 5 "https://www.digikey.de/product-detail/en/te-connectivity-amp-connectors/1734592-5/A101299CT-ND/2567441?utm_source=snapeda&utm_medium=aggregator&utm_campaign=symbol" H 6600 1600 50  0001 L BNN "Field5"
+F 6 "A101299CT-ND" H 6600 1600 50  0001 L BNN "Field6"
+F 7 "Compliant" H 6600 1600 50  0001 L BNN "Field7"
+F 8 "1734592-5" H 6600 1600 50  0001 L BNN "Field8"
+F 9 "https://www.te.com/usa-en/product-1734592-5.html?te_bu=Cor&te_type=disp&te_campaign=seda_glo_cor-seda-global-disp-prtnr-fy19-seda-model-bom-cta_sma-317_1&elqCampaignId=32493" H 6600 1600 50  0001 L BNN "Field9"
+F 10 "Conn FPC Connector SKT 5 POS 0.5mm Solder RA SMD T/R" H 6600 1600 50  0001 L BNN "Field10"
+F 11 "1734592-5" H 6600 1600 50  0001 L BNN "Field11"
+	1    6600 1600
+	-1   0    0    -1
+$EndComp
+$Comp
+L power:GND #PWR?
+U 1 1 5C996CA4
+P 6150 1950
+F 0 "#PWR?" H 6150 1700 50  0001 C CNN
+F 1 "GND" H 6155 1777 50  0000 C CNN
+F 2 "" H 6150 1950 50  0001 C CNN
+F 3 "" H 6150 1950 50  0001 C CNN
+	1    6150 1950
+	1    0    0    -1
+$EndComp
+Wire Wire Line
+	6200 1900 6150 1900
+Wire Wire Line
+	6150 1900 6150 1950
 $EndSCHEMATC

Commit message: minor changes to schematic and layout
Parts:
- gave numbers to parts that had none: 1
Other:
- note added: "GPIO Registers:\nPort 0 : P0.00 - P0.31\nPort 1 : P1.00 - P1.15"
Changed lines of the file:
@@
 $Descr A4 11693 8268
 encoding utf-8
-Sheet 2 3
+Sheet 2 4
 Title "nRF52840_breakout"
 Date "2019-03-22"
@@
 P 7550 2000
 AR Path="/5C9538B5" Ref="#PWR?"  Part="1"
-AR Path="/5C94F379/5C9538B5" Ref="#PWR031"  Part="1"
-F 0 "#PWR031" H 7550 1750 50  0001 C CNN
+AR Path="/5C94F379/5C9538B5" Ref="#PWR032"  Part="1"
+F 0 "#PWR032" H 7550 1750 50  0001 C CNN
 F 1 "GND" H 7555 1827 50  0000 C CNN
 F 2 "" H 7550 2000 50  0001 C CNN
@@
 NoConn ~ 950  2300
 $Comp
-L CONNECTOR_FFC_1734592-5:1734592-5 J?
+L CONNECTOR_FFC_1734592-5:1734592-5 J5
 U 1 1 5C986751
 P 6600 1600
-F 0 "J?" H 6372 1646 50  0000 R CNN
+F 0 "J5" H 6372 1646 50  0000 R CNN
 F 1 "1734592-5" H 6400 1550 50  0000 R CNN
 F 2 "custom_footprints:CONNECTOR_FFC_1734592-5" H 6600 1600 50  0001 L BNN
@@
 $EndComp
 $Comp
-L power:GND #PWR?
+L power:GND #PWR031
 U 1 1 5C996CA4
 P 6150 1950
-F 0 "#PWR?" H 6150 1700 50  0001 C CNN
+F 0 "#PWR031" H 6150 1700 50  0001 C CNN
 F 1 "GND" H 6155 1777 50  0000 C CNN
 F 2 "" H 6150 1950 50  0001 C CNN
@@
 Wire Wire Line
 	6150 1900 6150 1950
+Text Notes 650  6500 0    50   ~ 0
+GPIO Registers:\nPort 0 : P0.00 - P0.31\nPort 1 : P1.00 - P1.15
 $EndSCHEMATC

Commit message: added som like version of the breakout
Parts:
- removed C23, C24, C26: 10µF, Capacitor_SMD:C_0805_2012Metric_Pad1.15x1.40mm_HandSolder, symbol Device:C_Small
- removed C25: 100nF, Capacitor_SMD:C_0805_2012Metric_Pad1.15x1.40mm_HandSolder, symbol Device:C_Small
- removed C27: CTUNE1, Capacitor_SMD:C_0805_2012Metric_Pad1.15x1.40mm_HandSolder, symbol Device:C_Small
- removed C28: CTUNE2, Capacitor_SMD:C_0805_2012Metric_Pad1.15x1.40mm_HandSolder, symbol Device:C_Small
- removed D1: PRTR5V0U2X, Package_TO_SOT_SMD:SOT-143, symbol Power_Protection:PRTR5V0U2X
- removed FB1, FB2, FB3: 120R/0.55A, Inductor_SMD:L_0805_2012Metric_Pad1.15x1.40mm_HandSolder, symbol Device:Ferrite_Bead_Small
- removed H1, H2, H3, H4: MountingHole, MountingHole:MountingHole_2.2mm_M2_Pad_Via, symbol Mechanical:MountingHole
- removed J2, J3: Conn_01x12, Connector_PinHeader_2.54mm:PinHeader_1x12_P2.54mm_Vertical, symbol Connector_Generic:Conn_01x12
- removed J4: Conn_01x17, Connector_PinHeader_2.54mm:PinHeader_1x17_P2.54mm_Vertical, symbol Connector_Generic:Conn_01x17
- removed J5: 1734592-5, custom_footprints:CONNECTOR_FFC_1734592-5, symbol CONNECTOR_FFC_1734592-5:1734592-5
- removed J6: Pin Header 2x5, 1.27, Connector_PinHeader_1.27mm:PinHeader_2x05_P1.27mm_Vertical_SMD, symbol Connector_Generic:Conn_02x05_Odd_Even
- removed R1, R2: 5.1k, Resistor_SMD:R_0805_2012Metric_Pad1.15x1.40mm_HandSolder, symbol Device:R_Small
- removed R3, R4: 22, Resistor_SMD:R_0805_2012Metric_Pad1.15x1.40mm_HandSolder, symbol Device:R_Small
- removed TP1: VBUS_Raw, TestPoint:TestPoint_Pad_1.0x1.0mm, symbol Connector:TestPoint
- removed TP2: VBUS_nRF, TestPoint:TestPoint_Pad_1.0x1.0mm, symbol Connector:TestPoint
- removed TP3: NFC1, TestPoint:TestPoint_Pad_1.0x1.0mm, symbol Connector:TestPoint
- removed TP4: NFC2, TestPoint:TestPoint_Pad_1.0x1.0mm, symbol Connector:TestPoint
- removed U2: USB_TYPE_C, custom_footprints:USB_C_Receptacle_Amphenol_12401610E4-2A, symbol usb_type_c:USB_TYPE_C
- added J2: Conn_02x03_Odd_Even, Connector:Tag-Connect_TC2030-IDC-NL_2x03_P1.27mm_Vertical, symbol Connector_Generic:Conn_02x03_Odd_Even
- added J3, J5: Conn_01x22, Connector_PinHeader_1.27mm:PinHeader_1x22_P1.27mm_Vertical, symbol Connector_Generic:Conn_01x22
- added J4: Conn_01x16, Connector_PinHeader_1.27mm:PinHeader_1x16_P1.27mm_Vertical, symbol Connector_Generic:Conn_01x16
Connections:
- net labels added: VDDH, VDD_BAT
- net labels removed: VDIV
- wire segments 96 -> 10
- no-connect marks 15 -> 0
Other:
- note removed: "Connection Header"
- note removed: "GPIO Mapping"
- note removed: "Mounting Holes"
- note removed: "NFC Antenna Connector"
- note removed: "USB-C Connector"

Commit message: path selection/charging/bme680 sensor integration
Connections:
- net GND: now also J2.5 (Pin_5); no longer J2.4 (Pin_4)
- net P0.09_NFC1: now also J3.19 (Pin_19); no longer J3.18 (Pin_18)
- net P0.10_NFC2: now also J3.18 (Pin_18); no longer J3.19 (Pin_19)
- net P1.00_SWO: now also J2.6 (Pin_6); no longer J2.1 (Pin_1)
- net P1.18_RESET: now also J2.3 (Pin_3); no longer J2.2 (Pin_2)
- net SWDCLK: now also J2.4 (Pin_4); no longer J2.5 (Pin_5)
- net SWDIO: now also J2.2 (Pin_2); no longer J2.3 (Pin_3)
- net VDD_nRF: now also J2.1 (Pin_1); no longer J2.6 (Pin_6)
Changed lines of the file:
@@
 Comment4 ""
 $EndDescr
-Text GLabel 1650 1200 2    50   Input ~ 0
+Text GLabel 1150 1000 0    50   Input ~ 0
 VDD_nRF
 $Comp
 L power:GND #PWR?
 U 1 1 5C9538B5
-P 2150 1100
+P 1100 1250
 AR Path="/5C9538B5" Ref="#PWR?"  Part="1"
 AR Path="/5C94F379/5C9538B5" Ref="#PWR020"  Part="1"
-F 0 "#PWR020" H 2150 850 50  0001 C CNN
-F 1 "GND" H 2155 927 50  0000 C CNN
-F 2 "" H 2150 1100 50  0001 C CNN
-F 3 "" H 2150 1100 50  0001 C CNN
-	1    2150 1100
-	1    0    0    -1
-$EndComp
-Text GLabel 1150 1100 0    50   Input ~ 0
+F 0 "#PWR020" H 1100 1000 50  0001 C CNN
+F 1 "GND" H 1105 1077 50  0000 C CNN
+F 2 "" H 1100 1250 50  0001 C CNN
+F 3 "" H 1100 1250 50  0001 C CNN
+	1    1100 1250
+	1    0    0    -1
+$EndComp
+Text GLabel 1650 1000 2    50   Input ~ 0
 SWDIO
-Text GLabel 1150 1200 0    50   Input ~ 0
+Text GLabel 1650 1100 2    50   Input ~ 0
 SWDCLK
-Text GLabel 1650 1000 2    50   Input ~ 0
-P1.18_RESET
 Text Notes 600  600  0    50   ~ 0
 Debug IN Connector / Programmer
 Text Notes 7000 6850 0    50   ~ 0
 GPIO Registers:\nPort 0 : P0.00 - P0.31\nPort 1 : P1.00 - P1.15
-Text GLabel 1150 1000 0    50   Input ~ 0
-P1.00_SWO
 Text GLabel 6800 4700 0    50   Input ~ 0
 P0.12
@@
 Text GLabel 10500 4700 0    50   Input ~ 0
 P1.11
+Text GLabel 6800 4500 0    50   Input ~ 0
+P0.10_NFC2
 Text GLabel 6800 4400 0    50   Input ~ 0
-P0.10_NFC2
-Text GLabel 6800 4500 0    50   Input ~ 0
 P0.09_NFC1
 Text GLabel 10500 5900 0    50   Input ~ 0
@@
 	1    0    0    -1
 $EndComp
-Wire Wire Line
-	2150 1100 1650 1100
+Text GLabel 1650 1200 2    50   Input ~ 0
+P1.00_SWO
+Text GLabel 1150 1100 0    50   Input ~ 0
+P1.18_RESET
+Wire Wire Line
+	1150 1200 1100 1200
+Wire Wire Line
+	1100 1200 1100 1250
 $EndSCHEMATC
