File: nRF52840_breakout_power.sch (KiCad schematic (older format))
At the start: 12 parts, among them Q1 NTR1P02T1GOSTR-ND, U2 AP2112K-3.3, U3 MCP73831-2-OT

Commit message: modified bom / fixed silk,fab / added 3D models
Parts:
- added D3: LED_RED, LED_SMD:LED_0603_1608Metric, symbol Device:LED_Small
- added R6: 68R, Resistor_SMD:R_0402_1005Metric, symbol Device:R_Small
- C1, C2, C23: Description (none) -> CAP CER 10UF 6.3V X5R 0402; Digikey (none) -> 1276-1451-1-ND; LCSC (none) -> C15525; MFG P/N (none) -> CL05A106MQ5NUNC; Manufacturer (none) -> Samsung Electro-Mechanics
- D1: Description (none) -> DIODE SCHOTTKY 20V 1A SOD123FL; Digikey (none) -> MBR120VLSFT1GOSCT-ND; LCSC (none) -> C223608; MFG P/N (none) -> MBR120VLSFT1G; Manufacturer (none) -> ON Semiconductor
- D2: Description (none) -> LED ORANGE CLEAR CHIP SMD; Digikey 160-1445-2-ND -> 160-1434-1-ND; LCSC (none) -> C157740; MFG P/N LTST-C191KFKT -> LTST-C190KFKT; Manufacturer (none) -> Lite-On
- Q1: value NTR1P02T1GOSTR-ND -> pmos; Description (none) -> MOSFET P-CH 20V 1A SOT-23; LCSC (none) -> C129192; MFG P/N NTR1P02T1G -> NTR1P02T1G; Manufacturer (none) -> ON Semicon
- R1, R2: Description (none) -> RES SMD 100K OHM 5% 1/16W 0402; Digikey (none) -> 311-100KJRCT-ND; LCSC (none) -> C106234; MFG P/N (none) -> RC0402JR-07100KL; Manufacturer (none) -> Yageo
- R3: Description (none) -> RES SMD 2K OHM 1% 1/16W 0402; Digikey (none) -> 311-2KLRCT-ND; LCSC (none) -> C60488; MFG P/N (none) -> RC0402FR-072KL; Manufacturer (none) -> Yageo
- R4: Description (none) -> RES SMD 1K OHM 5% 1/16W 0402; Digikey (none) -> 311-1.0KJRCT-ND; LCSC (none) -> C105637; MFG P/N (none) -> RC0402JR-071KL; Manufacturer (none) -> Yageo
- U2: Description (none) -> IC REG LINEAR 3.3V 600MA SOT25; LCSC (none) -> C51118; MFG P/N AP2112K-3.3TRG1 -> AP2112K-3.3TRG1; Manufacturer (none) -> Diodes Incorporated
- U3: Description (none) -> IC CONTROLLR LI-ION 4.2V SOT23-5; Digikey MCP73831T-2ACI/OTCT-ND -> MCP73831T-2ATI/OTCT-ND; LCSC (none) -> C14879; MFG P/N MCP73831T-2ACI/OT -> MCP73831T-2ATI/OT; Manufacturer (none) -> Microchip Tech
Connections:
- net GND: now also D3.1 (K)
- net VDD_nRF: now also R6.1
- new net: D3.2 (A), R6.2
Changed lines of the file:
@@
 F 1 "100k" H 859 1655 50  0000 L CNN
 F 2 "Resistor_SMD:R_0402_1005Metric" H 800 1700 50  0001 C CNN
-F 3 "~" H 800 1700 50  0001 C CNN
+F 3 "http://www.yageo.com/documents/recent/PYu-RC_Group_51_RoHS_L_10.pdf" H 800 1700 50  0001 C CNN
+F 4 " RES SMD 100K OHM 5% 1/16W 0402 " H 800 1700 50  0001 C CNN "Description"
+F 5 " 311-100KJRCT-ND " H 800 1700 50  0001 C CNN "Digikey"
+F 6 "C106234" H 800 1700 50  0001 C CNN "LCSC"
+F 7 "RC0402JR-07100KL" H 800 1700 50  0001 C CNN "MFG P/N"
+F 8 "Yageo" H 800 1700 50  0001 C CNN "Manufacturer"
 	1    800  1700
 	1    0    0    -1
@@
 F 1 "MBR120" H 1050 1436 50  0000 C CNN
 F 2 "Diode_SMD:D_SOD-123" V 1050 1550 50  0001 C CNN
-F 3 "~" V 1050 1550 50  0001 C CNN
+F 3 "https://www.onsemi.com/pub/Collateral/MBR120VLSFT1-D.PDF" V 1050 1550 50  0001 C CNN
+F 4 " DIODE SCHOTTKY 20V 1A SOD123FL " H 1050 1550 50  0001 C CNN "Description"
+F 5 " MBR120VLSFT1GOSCT-ND " H 1050 1550 50  0001 C CNN "Digikey"
+F 6 "C223608" H 1050 1550 50  0001 C CNN "LCSC"
+F 7 " MBR120VLSFT1G " H 1050 1550 50  0001 C CNN "MFG P/N"
+F 8 "ON Semiconductor" H 1050 1550 50  0001 C CNN "Manufacturer"
 	1    1050 1550
 	-1   0    0    1
@@
 F 1 "10uF" H 1342 1655 50  0000 L CNN
 F 2 "Capacitor_SMD:C_0402_1005Metric" H 1250 1700 50  0001 C CNN
-F 3 "~" H 1250 1700 50  0001 C CNN
+F 3 "https://media.digikey.com/pdf/Data%20Sheets/Samsung%20PDFs/CL_Series_MLCC_ds.pdf" H 1250 1700 50  0001 C CNN
+F 4 " CAP CER 10UF 6.3V X5R 0402 " H 1250 1700 50  0001 C CNN "Description"
+F 5 " 1276-1451-1-ND " H 1250 1700 50  0001 C CNN "Digikey"
+F 6 "C15525" H 1250 1700 50  0001 C CNN "LCSC"
+F 7 " CL05A106MQ5NUNC " H 1250 1700 50  0001 C CNN "MFG P/N"
+F 8 "Samsung Electro-Mechanics" H 1250 1700 50  0001 C CNN "Manufacturer"
 	1    1250 1700
 	1    0    0    -1
@@
 F 2 "Package_TO_SOT_SMD:SOT-23-5" H 2400 1975 50  0001 C CNN
 F 3 "https://www.diodes.com/assets/Datasheets/AP2112.pdf" H 2400 1750 50  0001 C CNN
-F 4 " AP2112K-3.3TRG1 " H 2400 1650 50  0001 C CNN "MFG P/N"
+F 4 "AP2112K-3.3TRG1 " H 2400 1650 50  0001 C CNN "MFG P/N"
 F 5 " AP2112K-3.3TRG1DICT-ND " H 2400 1650 50  0001 C CNN "Digikey"
+F 6 " IC REG LINEAR 3.3V 600MA SOT25 " H 2400 1650 50  0001 C CNN "Description"
+F 7 "C51118" H 2400 1650 50  0001 C CNN "LCSC"
+F 8 "Diodes Incorporated" H 2400 1650 50  0001 C CNN "Manufacturer"
 	1    2400 1650
 	1    0    0    -1
@@
 F 1 "100k" V 2050 1650 50  0000 C CNN
 F 2 "Resistor_SMD:R_0402_1005Metric" H 1950 1650 50  0001 C CNN
-F 3 "~" H 1950 1650 50  0001 C CNN
+F 3 "http://www.yageo.com/documents/recent/PYu-RC_Group_51_RoHS_L_10.pdf" H 1950 1650 50  0001 C CNN
+F 4 " RES SMD 100K OHM 5% 1/16W 0402 " H 1950 1650 50  0001 C CNN "Description"
+F 5 " 311-100KJRCT-ND " H 1950 1650 50  0001 C CNN "Digikey"
+F 6 "C106234" H 1950 1650 50  0001 C CNN "LCSC"
+F 7 "RC0402JR-07100KL" H 1950 1650 50  0001 C CNN "MFG P/N"
+F 8 "Yageo" H 1950 1650 50  0001 C CNN "Manufacturer"
 	1    1950 1650
 	0    1    1    0
@@
 F 1 "10uF" H 2892 1655 50  0000 L CNN
 F 2 "Capacitor_SMD:C_0402_1005Metric" H 2800 1700 50  0001 C CNN
-F 3 "~" H 2800 1700 50  0001 C CNN
+F 3 "https://media.digikey.com/pdf/Data%20Sheets/Samsung%20PDFs/CL_Series_MLCC_ds.pdf" H 2800 1700 50  0001 C CNN
+F 4 " CAP CER 10UF 6.3V X5R 0402 " H 2800 1700 50  0001 C CNN "Description"
+F 5 " 1276-1451-1-ND " H 2800 1700 50  0001 C CNN "Digikey"
+F 6 "C15525" H 2800 1700 50  0001 C CNN "LCSC"
+F 7 " CL05A106MQ5NUNC " H 2800 1700 50  0001 C CNN "MFG P/N"
+F 8 "Samsung Electro-Mechanics" H 2800 1700 50  0001 C CNN "Manufacturer"
 	1    2800 1700
 	1    0    0    -1
@@
 F 2 "Package_TO_SOT_SMD:SOT-23-5" H 8050 1550 50  0001 L CIN
 F 3 "http://ww1.microchip.com/downloads/en/DeviceDoc/20001984g.pdf" H 7850 1750 50  0001 C CNN
-F 4 " MCP73831T-2ACI/OTCT-ND " H 8000 1800 50  0001 C CNN "Digikey"
-F 5 " MCP73831T-2ACI/OT " H 8000 1800 50  0001 C CNN "MFG P/N"
+F 4 " MCP73831T-2ATI/OTCT-ND " H 8000 1800 50  0001 C CNN "Digikey"
+F 5 "MCP73831T-2ATI/OT" H 8000 1800 50  0001 C CNN "MFG P/N"
+F 6 " IC CONTROLLR LI-ION 4.2V SOT23-5 " H 8000 1800 50  0001 C CNN "Description"
+F 7 "C14879" H 8000 1800 50  0001 C CNN "LCSC"
+F 8 "Microchip Tech" H 8000 1800 50  0001 C CNN "Manufacturer"
 	1    8000 1800
 	1    0    0    -1
@@
 F 1 "LED_ORG" H 7500 2436 50  0000 C CNN
 F 2 "LED_SMD:LED_0603_1608Metric" V 7500 2550 50  0001 C CNN
-F 3 "http://optoelectronics.liteon.com/upload/download/DS22-2000-222/LTST-C191KFKT.pdf" V 7500 2550 50  0001 C CNN
-F 4 " LTST-C191KFKT " H 7500 2550 50  0001 C CNN "MFG P/N"
-F 5 " 160-1445-2-ND " H 7500 2550 50  0001 C CNN "Digikey"
+F 3 "http://optoelectronics.liteon.com/upload/download/DS-22-99-0186/LTST-C190KFKT.PDF" V 7500 2550 50  0001 C CNN
+F 4 "LTST-C190KFKT" H 7500 2550 50  0001 C CNN "MFG P/N"
+F 5 " 160-1434-1-ND " H 7500 2550 50  0001 C CNN "Digikey"
+F 6 " LED ORANGE CLEAR CHIP SMD " H 7500 2550 50  0001 C CNN "Description"
+F 7 "Lite-On" H 7500 2550 50  0001 C CNN "Manufacturer"
+F 8 "C157740" H 7500 2550 50  0001 C CNN "LCSC"
 	1    7500 2550
 	-1   0    0    1
@@
 F 1 "1k" V 7795 2550 50  0000 C CNN
 F 2 "Resistor_SMD:R_0402_1005Metric" H 7900 2550 50  0001 C CNN
-F 3 "~" H 7900 2550 50  0001 C CNN
+F 3 "http://www.yageo.com/documents/recent/PYu-RC_Group_51_RoHS_L_10.pdf" H 7900 2550 50  0001 C CNN
+F 4 " RES SMD 1K OHM 5% 1/16W 0402 " H 7900 2550 50  0001 C CNN "Description"
+F 5 " 311-1.0KJRCT-ND " H 7900 2550 50  0001 C CNN "Digikey"
+F 6 "C105637" H 7900 2550 50  0001 C CNN "LCSC"
+F 7 "RC0402JR-071KL" H 7900 2550 50  0001 C CNN "MFG P/N"
+F 8 "Yageo" H 7900 2550 50  0001 C CNN "Manufacturer"
 	1    7900 2550
 	0    1    1    0
@@
 F 1 "2k" V 7395 2200 50  0000 C CNN
 F 2 "Resistor_SMD:R_0402_1005Metric" H 7500 2200 50  0001 C CNN
-F 3 "~" H 7500 2200 50  0001 C CNN
+F 3 "http://www.yageo.com/documents/recent/PYu-RC_Group_51_RoHS_L_10.pdf" H 7500 2200 50  0001 C CNN
+F 4 " RES SMD 2K OHM 1% 1/16W 0402 " H 7500 2200 50  0001 C CNN "Description"
+F 5 " 311-2KLRCT-ND " H 7500 2200 50  0001 C CNN "Digikey"
+F 6 "C60488" H 7500 2200 50  0001 C CNN "LCSC"
+F 7 "RC0402FR-072KL" H 7500 2200 50  0001 C CNN "MFG P/N"
+F 8 "Yageo" H 7500 2200 50  0001 C CNN "Manufacturer"
 	1    7500 2200
 	0    1    1    0
@@
 F 1 "10uF" H 8742 1805 50  0000 L CNN
 F 2 "Capacitor_SMD:C_0402_1005Metric" H 8650 1850 50  0001 C CNN
-F 3 "~" H 8650 1850 50  0001 C CNN
+F 3 "https://media.digikey.com/pdf/Data%20Sheets/Samsung%20PDFs/CL_Series_MLCC_ds.pdf" H 8650 1850 50  0001 C CNN
+F 4 " CAP CER 10UF 6.3V X5R 0402 " H 8650 1850 50  0001 C CNN "Description"
+F 5 " 1276-1451-1-ND " H 8650 1850 50  0001 C CNN "Digikey"
+F 6 "C15525" H 8650 1850 50  0001 C CNN "LCSC"
+F 7 " CL05A106MQ5NUNC " H 8650 1850 50  0001 C CNN "MFG P/N"
+F 8 "Samsung Electro-Mechanics" H 8650 1850 50  0001 C CNN "Manufacturer"
 	1    8650 1850
 	1    0    0    -1
@@
 P 1150 1150
 F 0 "Q1" H 1356 1196 50  0000 L CNN
-F 1 " NTR1P02T1GOSTR-ND " H 1356 1105 50  0000 L CNN
+F 1 "pmos" H 1356 1105 50  0000 L CNN
 F 2 "Package_TO_SOT_SMD:SOT-23" H 1350 1250 50  0001 C CNN
 F 3 "https://www.onsemi.com/pub/Collateral/NTR1P02T1-D.PDF" H 1150 1150 50  0001 C CNN
-F 4 " NTR1P02T1G " H 1150 1150 50  0001 C CNN "MFG P/N"
+F 4 "NTR1P02T1G" H 1150 1150 50  0001 C CNN "MFG P/N"
 F 5 " NTR1P02T1GOSTR-ND " H 1150 1150 50  0001 C CNN "Digikey"
+F 6 " MOSFET P-CH 20V 1A SOT-23 " H 1150 1150 50  0001 C CNN "Description"
+F 7 "C129192" H 1150 1150 50  0001 C CNN "LCSC"
+F 8 "ON Semicon" H 1150 1150 50  0001 C CNN "Manufacturer"
 	1    1150 1150
 	1    0    0    -1
 $EndComp
+Text GLabel 4700 1450 2    50   Input ~ 0
+VDD_nRF
+$Comp
+L Device:R_Small R6
+U 1 1 5D3752EE
+P 4700 1700
+F 0 "R6" H 4759 1746 50  0000 L CNN
+F 1 "68R" H 4759 1655 50  0000 L CNN
+F 2 "Resistor_SMD:R_0402_1005Metric" H 4700 1700 50  0001 C CNN
+F 3 "http://www.yageo.com/NewPortal/yageodocoutput?fileName=/pdf/R-Chip/PYu-AC_51_RoHS_L_6.pdf" H 4700 1700 50  0001 C CNN
+F 4 " RES SMD 68 OHM 1% 1/16W 0402 " H 4700 1700 50  0001 C CNN "Description"
+F 5 " YAG3507CT-ND " H 4700 1700 50  0001 C CNN "Digikey"
+F 6 "C227192" H 4700 1700 50  0001 C CNN "LCSC"
+F 7 "AC0402FR-0768RL" H 4700 1700 50  0001 C CNN "MFG P/N"
+F 8 "Yageo" H 4700 1700 50  0001 C CNN "Manufacturer"
+	1    4700 1700
+	1    0    0    -1
+$EndComp
+$Comp
+L power:GND #PWR0108
+U 1 1 5D375800
+P 4700 2100
+F 0 "#PWR0108" H 4700 1850 50  0001 C CNN
+F 1 "GND" H 4705 1927 50  0000 C CNN
+F 2 "" H 4700 2100 50  0001 C CNN
+F 3 "" H 4700 2100 50  0001 C CNN
+	1    4700 2100
+	1    0    0    -1
+$EndComp
+Wire Wire Line
+	4700 1450 4700 1600
+Wire Wire Line
+	4700 1800 4700 1850
+Wire Wire Line
+	4700 2050 4700 2100
+$Comp
+L Device:LED_Small D3
+U 1 1 5D3794D0
+P 4700 1950
+F 0 "D3" V 4746 1882 50  0000 R CNN
+F 1 "LED_RED" V 4655 1882 50  0000 R CNN
+F 2 "LED_SMD:LED_0603_1608Metric" V 4700 1950 50  0001 C CNN
+F 3 "http://optoelectronics.liteon.com/upload/download/DS22-2000-223/LTST-C191KRKT.PDF" V 4700 1950 50  0001 C CNN
+F 4 " LED RED CLEAR SMD " H 4700 1950 50  0001 C CNN "Description"
+F 5 " 160-1447-1-ND " H 4700 1950 50  0001 C CNN "Digikey"
+F 6 "C125099" H 4700 1950 50  0001 C CNN "LCSC"
+F 7 "LTST-C191KRKT" H 4700 1950 50  0001 C CNN "MFG P/N"
+F 8 "Lite-On" H 4700 1950 50  0001 C CNN "Manufacturer"
+	1    4700 1950
+	0    -1   -1   0
+$EndComp
 $EndSCHEMATC
